File: v1/line_follower.kicad_pcb (KiCad board)
At the start: 2 copper layers, 60 x 80 mm, 25 parts, among them K1 BUZZER, P1 QTR-8A, P2 HC-05, P3 EXP HEADER, P4 LEFT MOTOR, P5 RIGHT MOTOR, P6 BATTERY, SW1 SW_PUSH, SW2 SW_PUSH, SW3 SW_PUSH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

Commit message: Add missing graphics and mounting holes
Parts:
- added G***: LOGO, line_follower:osh_logo, F.Cu at (133.2, 92.2)
- added G***: LOGO, line_follower:bug_a_logo, F.Cu at (133.5, 80.2)
- added G***: LOGO, line_follower:cc_by_sa_logo, F.Cu at (174.8, 99.2)
- added Ref**: MountingHole_3mm, line_follower:MountingHole_3mm, F.Cu at (122.0, 63.0)
- added Ref**: MountingHole_3mm, line_follower:MountingHole_3mm, F.Cu at (174.0, 63.0)
- added Ref**: MountingHole_3mm, line_follower:MountingHole_3mm, F.Cu at (122.0, 135.0)
- added Ref**: MountingHole_3mm, line_follower:MountingHole_3mm, F.Cu at (174.0, 135.0)
